File: uSD-Turbo.kicad_pcb (KiCad board)
At the start: 2 copper layers, 32.4 x 25.5 mm, 14 parts, among them J1 User Port, U1 74LVC125AD, U2 AMS1117-3.3

Commit message: Renamed project, added resistor between PB1 and CB1, added BOM and Gerber files
Parts:
- added R5: 56 Ω, Resistor_SMD:R_0603_1608Metric, F.Cu at (113.0, 63.7)
- moved C5 4.49 mm to (120.6, 67.8), turned to 90 degrees
- moved C1 2.79 mm to (116.8, 62.9)
- moved C2 2.79 mm to (116.8, 64.5)
Connections:
- J1 pad 2: unconnected-(J1-Pin_2-Pad2) -> CB1
Routing:
- net PB1: track 19.2 -> 30.3 mm, vias 2 -> 3
- net CB1: track 0.00 -> 6.47 mm
- net +3.3V: track 51.0 -> 48.2 mm
- net GND: track 39.0 -> 36.5 mm, vias 18 -> 17
- net +5V: track 10.7 -> 12.3 mm
Other:
- board text added: "J. Hilsdorf µSD Turbo 1.0"
- board text removed: "Jan Hilsdorf 07/2023"
